File: GDC0689.sch (KiCad schematic (older format))
At the start: 10 parts, among them P1 CONN_01X03, P2 CONN_01X07, P3 CONN_01X02, P4 CONN_01X02, Y1 Crystal

Commit message: Add link
Connections:
- wire segments 100 -> 102
- no-connect marks 8 -> 7
Changed lines of the file:
@@
 	1    0    0    -1
 $EndComp
-Wire Wire Line
-	4650 3150 4150 3100
-Wire Wire Line
-	4150 3200 4650 3250
-Wire Wire Line
-	4300 3350 4650 3350
-Wire Wire Line
-	4300 3450 4650 3450
-Wire Wire Line
-	4300 3550 4650 3550
-Wire Wire Line
-	4300 3650 4650 3650
-Wire Wire Line
-	4400 4300 4800 4300
-Wire Wire Line
-	4400 4400 4800 4400
-Wire Wire Line
-	4400 4500 4800 4500
-Wire Wire Line
-	4400 4600 4800 4600
-Wire Wire Line
-	4200 1350 4650 1350
-Wire Wire Line
-	4650 1450 4200 1450
-Wire Wire Line
-	4650 1550 4200 1550
-Wire Wire Line
-	4200 1650 4650 1650
-Wire Wire Line
-	4650 1750 4200 1750
-Wire Wire Line
-	4200 1850 4650 1850
-Wire Wire Line
-	4200 1950 4650 1950
-Wire Wire Line
-	4200 2050 4650 2050
-Wire Wire Line
-	4200 5700 4800 5700
-Wire Wire Line
-	4200 5600 4800 5600
-Wire Wire Line
-	4200 5500 4800 5500
-Wire Wire Line
-	4200 5400 4800 5400
-Wire Wire Line
-	4200 5300 4800 5300
-Wire Wire Line
-	4200 5200 4800 5200
-Wire Wire Line
-	4200 5100 4800 5100
-Wire Wire Line
-	4200 5000 4800 5000
-Wire Wire Line
-	4800 4700 4600 4700
-Wire Wire Line
-	4800 4800 4600 4800
-Wire Wire Line
-	4800 4900 4600 4900
-Wire Wire Line
-	6050 1350 6250 1350
-Wire Wire Line
-	6050 1450 6250 1450
-Wire Wire Line
-	6050 1550 6250 1550
-Wire Wire Line
-	6050 1650 6350 1650
-Wire Wire Line
-	6050 1750 6350 1750
-Wire Wire Line
-	6050 1850 6350 1850
-Wire Wire Line
-	6050 1950 6350 1950
-Wire Wire Line
-	6050 2050 6350 2050
-Wire Wire Line
-	6050 2150 6350 2150
-Wire Wire Line
-	6050 2250 6350 2250
-Wire Wire Line
-	6050 2350 6350 2350
-Wire Wire Line
-	6050 2450 6350 2450
-Wire Wire Line
-	6050 2550 6350 2550
-Wire Wire Line
-	6050 2650 6350 2650
-Wire Wire Line
-	6050 2750 6350 2750
-Wire Wire Line
-	6050 2850 6350 2850
-Wire Wire Line
-	6050 2950 6350 2950
-Wire Wire Line
-	6000 4350 6250 4350
-Wire Wire Line
-	6000 4450 6250 4450
-Wire Wire Line
-	6000 4550 6250 4550
-Wire Wire Line
-	6000 4650 6250 4650
-Wire Wire Line
-	6000 4750 6250 4750
-Wire Wire Line
-	6000 4850 6250 4850
-Wire Wire Line
-	6000 4950 6250 4950
-Wire Wire Line
-	6000 5050 6250 5050
-Wire Wire Line
-	6000 5150 6250 5150
-Wire Wire Line
-	6000 5250 6250 5250
-Wire Wire Line
-	6000 5350 6250 5350
-Wire Wire Line
-	6000 5450 6250 5450
-Wire Wire Line
-	6000 5550 6250 5550
-Wire Wire Line
-	6000 5650 6250 5650
-Wire Wire Line
-	4650 2550 4100 2550
-Wire Wire Line
-	1500 3750 1500 3650
-Wire Wire Line
-	1500 3650 2200 3650
-Wire Wire Line
-	1500 3850 1500 3950
-Wire Wire Line
-	1500 3950 2200 3950
-Wire Wire Line
-	4650 2850 4350 2850
-Wire Wire Line
-	4650 2750 4350 2750
-Wire Wire Line
-	4650 2650 4350 2650
-Wire Wire Line
-	4650 2950 4350 2950
-Wire Wire Line
-	1500 2000 1800 2000
-Wire Wire Line
-	1500 2100 2400 2100
-Wire Wire Line
-	1900 1750 1800 1750
-Wire Wire Line
-	1800 1750 1800 2000
-Wire Wire Line
-	1500 2200 1950 2200
-Wire Wire Line
-	1500 2300 1950 2300
-Wire Wire Line
-	1500 2400 1950 2400
-Wire Wire Line
-	1500 2500 1950 2500
-Wire Wire Line
-	1500 2600 1950 2600
-Wire Wire Line
-	4650 2150 4300 2150
-Wire Wire Line
-	4650 2250 4300 2250
-Wire Wire Line
-	4650 2350 4300 2350
-Wire Wire Line
-	4650 2450 4300 2450
-Wire Wire Line
-	4650 3050 4350 3050
-Wire Wire Line
-	1500 2950 2050 2950
-Wire Wire Line
-	1500 3050 1750 3050
-Connection ~ 1800 3950
-Connection ~ 1800 3650
-Connection ~ 1800 2100
 Text Label 1800 2100 2    60   ~ 0
 VCC
-Connection ~ 4100 2550
-Connection ~ 2100 2100
-Wire Wire Line
-	1750 3050 1750 3250
 $Comp
 L R R3
@@
 	0    1    1    0
 $EndComp
-Wire Wire Line
-	5100 6000 5300 6000
-Wire Wire Line
-	2950 6000 4800 6000
 $Comp
 L GNDREF #PWR04
@@
 	1    0    0    -1
 $EndComp
-Wire Wire Line
-	5500 6000 5500 6100
-Connection ~ 2400 2100
 $Comp
 L PWR_FLAG #FLG05
@@
 	1    0    0    -1
 $EndComp
-Connection ~ 1800 1750
-Connection ~ 5300 6000
-Connection ~ 4550 6000
-Wire Wire Line
-	2950 6000 2950 1800
-Wire Wire Line
-	2950 1800 2100 1800
-Connection ~ 5100 6000
-Connection ~ 4800 6000
 Text Label 4350 3350 0    60   ~ 0
 COM1
-Wire Wire Line
-	2500 2600 2100 2600
 $Comp
 L R R1
@@
 	1    0    0    -1
 $EndComp
-Wire Wire Line
-	2100 1800 2100 2200
-Wire Wire Line
-	2100 2600 2100 2500
 $Comp
 L CONN_01X03 P1
@@
 	-1   0    0    1
 $EndComp
-Wire Wire Line
-	1500 3750 1300 3750
-Wire Wire Line
-	1500 3850 1300 3850
-Wire Wire Line
-	1300 3950 1300 4100
-Wire Wire Line
-	1300 4100 1500 4100
 $Comp
 L GNDREF #PWR07
@@
 $EndComp
 Wire Wire Line
+	4650 3150 4150 3100
+Wire Wire Line
+	4150 3200 4650 3250
+Wire Wire Line
+	4300 3350 4650 3350
+Wire Wire Line
+	4300 3450 4650 3450
+Wire Wire Line
+	4300 3550 4650 3550
+Wire Wire Line
+	4300 3650 4650 3650
+Wire Wire Line
+	4400 4300 4800 4300
+Wire Wire Line
+	4400 4400 4800 4400
+Wire Wire Line
+	4400 4500 4800 4500
+Wire Wire Line
+	4400 4600 4800 4600
+Wire Wire Line
+	4200 1350 4650 1350
+Wire Wire Line
+	4650 1450 4200 1450
+Wire Wire Line
+	4650 1550 4200 1550
+Wire Wire Line
+	4200 1650 4650 1650
+Wire Wire Line
+	4650 1750 4200 1750
+Wire Wire Line
+	4200 1850 4650 1850
+Wire Wire Line
+	4200 1950 4650 1950
+Wire Wire Line
+	4200 2050 4650 2050
+Wire Wire Line
+	4200 5700 4800 5700
+Wire Wire Line
+	4200 5600 4800 5600
+Wire Wire Line
+	4200 5500 4800 5500
+Wire Wire Line
+	4200 5400 4800 5400
+Wire Wire Line
+	4200 5300 4800 5300
+Wire Wire Line
+	4200 5200 4800 5200
+Wire Wire Line
+	4200 5100 4800 5100
+Wire Wire Line
+	4200 5000 4800 5000
+Wire Wire Line
+	4800 4700 4600 4700
+Wire Wire Line
+	4800 4800 4600 4800
+Wire Wire Line
+	4800 4900 4600 4900
+Wire Wire Line
+	6050 1350 6250 1350
+Wire Wire Line
+	6050 1450 6250 1450
+Wire Wire Line
+	6050 1550 6250 1550
+Wire Wire Line
+	6050 1650 6350 1650
+Wire Wire Line
+	6050 1750 6350 1750
+Wire Wire Line
+	6050 1850 6350 1850
+Wire Wire Line
+	6050 1950 6350 1950
+Wire Wire Line
+	6050 2050 6350 2050
+Wire Wire Line
+	6050 2150 6350 2150
+Wire Wire Line
+	6050 2250 6350 2250
+Wire Wire Line
+	6050 2350 6350 2350
+Wire Wire Line
+	6050 2450 6350 2450
+Wire Wire Line
+	6050 2550 6350 2550
+Wire Wire Line
+	6050 2650 6350 2650
+Wire Wire Line
+	6050 2750 6350 2750
+Wire Wire Line
+	6050 2850 6350 2850
+Wire Wire Line
+	6050 2950 6350 2950
+Wire Wire Line
+	6000 4350 6250 4350
+Wire Wire Line
+	6000 4450 6250 4450
+Wire Wire Line
+	6000 4550 6250 4550
+Wire Wire Line
+	6000 4650 6250 4650
+Wire Wire Line
+	6000 4750 6250 4750
+Wire Wire Line
+	6000 4850 6250 4850
+Wire Wire Line
+	6000 4950 6250 4950
+Wire Wire Line
+	6000 5050 6250 5050
+Wire Wire Line
+	6000 5150 6250 5150
+Wire Wire Line
+	6000 5250 6250 5250
+Wire Wire Line
+	6000 5350 6250 5350
+Wire Wire Line
+	6000 5450 6250 5450
+Wire Wire Line
+	6000 5550 6250 5550
+Wire Wire Line
+	6000 5650 6250 5650
+Wire Wire Line
+	4650 2550 4100 2550
+Wire Wire Line
+	1500 3750 1500 3650
+Wire Wire Line
+	1500 3650 2200 3650
+Wire Wire Line
+	1500 3850 1500 3950
+Wire Wire Line
+	1500 3950 2200 3950
+Wire Wire Line
+	4650 2850 4350 2850
+Wire Wire Line
+	4650 2750 4350 2750
+Wire Wire Line
+	4650 2650 4350 2650
+Wire Wire Line
+	4650 2950 4350 2950
+Wire Wire Line
+	1500 2000 1800 2000
+Wire Wire Line
+	1500 2100 2400 2100
+Wire Wire Line
+	1900 1750 1800 1750
+Wire Wire Line
+	1800 1750 1800 2000
+Wire Wire Line
+	1500 2200 1950 2200
+Wire Wire Line
+	1500 2300 1950 2300
+Wire Wire Line
+	1500 2400 1950 2400
+Wire Wire Line
+	1500 2500 1950 2500
+Wire Wire Line
+	1500 2600 1950 2600
+Wire Wire Line
+	4650 2150 4300 2150
+Wire Wire Line
+	4650 2250 4300 2250
+Wire Wire Line
+	4650 2350 4300 2350
+Wire Wire Line
+	4650 2450 4300 2450
+Wire Wire Line
+	4650 3050 4350 3050
+Wire Wire Line
+	1500 2950 2050 2950
+Wire Wire Line
+	1500 3050 1750 3050
+Connection ~ 1800 3950
+Connection ~ 1800 3650
+Connection ~ 1800 2100
+Connection ~ 4100 2550
+Connection ~ 2100 2100
+Wire Wire Line
+	1750 3050 1750 3250
+Wire Wire Line
+	5100 6000 5300 6000
+Wire Wire Line
+	2950 6000 4800 6000
+Wire Wire Line
+	5500 6000 5500 6100
+Connection ~ 2400 2100
+Connection ~ 1800 1750
+Connection ~ 5300 6000
+Connection ~ 4550 6000
+Wire Wire Line
+	2950 6000 2950 1800
+Wire Wire Line
+	2950 1800 2100 1800
+Connection ~ 5100 6000
+Connection ~ 4800 6000
+Wire Wire Line
+	2500 2600 2100 2600
+Wire Wire Line
+	2100 1800 2100 2200
+Wire Wire Line
+	2100 2600 2100 2500
+Wire Wire Line
+	1500 3750 1300 3750
+Wire Wire Line
+	1500 3850 1300 3850
+Wire Wire Line
+	1300 3950 1300 4100
+Wire Wire Line
+	1300 4100 1500 4100
+Wire Wire Line
 	2360 2850 2360 3250
 Wire Wire Line
 	2360 3250 1750 3250
-NoConn ~ 2500 3100
+Wire Wire Line
+	2500 3100 2360 3100
+Wire Wire Line
+	2360 3100 2360 3105
+Connection ~ 2360 3105
 $EndSCHEMATC
